File: Schematics/sensor-hub/hub-peripherals.kicad_sch (KiCad schematic)
At the start: 17 parts

Commit message: schematic and pcb upload
Parts:
- removed C?: 0.1uf, symbol Device:C
- removed C? (x4): 0.1u, symbol Device:C
- removed R? (x4): 4.7k, symbol Device:R
- removed SW? (x4): SW_Push, symbol Switch:SW_Push
- removed U?: CR2013-MI2120, Display:CR2013-MI2120, symbol Driver_Display:CR2013-MI2120
- added C14, C15, C16, C17: 1n, Capacitor_SMD:C_0805_2012Metric_Pad1.18x1.45mm_HandSolder, symbol Device:C
- added J3: Conn_01x09_Male, Connector_PinHeader_2.54mm:PinHeader_1x09_P2.54mm_Vertical, symbol Connector:Conn_01x09_Male
- added R16, R17, R18, R19, R20, R21, R22, R23, R24: 10k, Resistor_SMD:R_0805_2012Metric_Pad1.20x1.40mm_HandSolder, symbol Device:R
- added SW4, SW5, SW6, SW7: SW_Push, Button_Switch_THT:SW_PUSH-12mm, symbol Switch:SW_Push
- C13: renamed from C?; value 0.1u -> 1n; footprint (none) -> Capacitor_SMD:C_0805_2012Metric_Pad1.18x1.45mm_HandSolder
- R15: renamed from R?; value 4.7k -> 10k; footprint (none) -> Resistor_SMD:R_0805_2012Metric_Pad1.20x1.40mm_HandSolder
- SW3: renamed from SW?; footprint (none) -> Button_Switch_THT:SW_PUSH-12mm
Connections:
- net +3V3: now also J3.1 (Pin_1), SW4.1, SW5.1, SW6.1, SW7.1; no longer C13.2
- net GND: now also C14.1, C15.1, C16.1, C17.1, J3.2 (Pin_2), R16.1, R17.1, R18.1, R19.1
- net SWITCH0: now also C13.2, R20.1; no longer R15.2, SW3.2
- net SWITCH1: now also C14.2, R21.1
- net SWITCH2: now also C15.2, R22.1
- net SWITCH3: now also C16.2, R23.1
- net SWITCH4: now also C17.2, R24.1
- new net: R18.2, R23.2, SW6.2
- new net: R16.2, R21.2, SW4.2
- new net: R15.2, R20.2, SW3.2
- new net: R17.2, R22.2, SW5.2
- new net: R19.2, R24.2, SW7.2
- new net DISP.CS: J3.3 (Pin_3)
- new net DISP.DC: J3.5 (Pin_5)
- new net DISP.LED: J3.8 (Pin_8)
- new net DISP.RESET: J3.4 (Pin_4)
- new net DISP.SCK: J3.7 (Pin_7)
- new net DISP.SDI: J3.6 (Pin_6)
- new net DISP.SDO: J3.9 (Pin_9)
- no-connect marks 5 -> 0
Other:
- note added: "Display Module Pins"
- note removed: "Display Module"
- moved on the sheet: C13, R15, SW3
