File: Schematics/sensor-hub/hub-usb-pwr.kicad_sch (KiCad schematic)
At the start: 15 parts

Commit message: schematic and pcb upload
Parts:
- removed D?: LED, symbol Device:LED
- removed R?: 150, symbol Device:R
- added C1, C6: 1u, Capacitor_SMD:C_0805_2012Metric_Pad1.18x1.45mm_HandSolder, symbol Device:C
- added C2: 4.7u, Capacitor_SMD:C_0805_2012Metric_Pad1.18x1.45mm_HandSolder, symbol Device:C
- added C5: 0.1u, Capacitor_SMD:C_0805_2012Metric_Pad1.18x1.45mm_HandSolder, symbol Device:C
- added D3, D4: LED, LED_SMD:LED_0805_2012Metric_Pad1.15x1.40mm_HandSolder, symbol Device:LED
- added J2: Conn_01x03, Connector_JST:JST_PH_B3B-PH-K_1x03_P2.00mm_Vertical, symbol Connector_Generic:Conn_01x03
- added R1: 4.12k, Resistor_SMD:R_0805_2012Metric_Pad1.20x1.40mm_HandSolder, symbol Device:R
- added R2: 1.18k, Resistor_SMD:R_0805_2012Metric_Pad1.20x1.40mm_HandSolder, symbol Device:R
- added R3: 1.13k, Resistor_SMD:R_0805_2012Metric_Pad1.20x1.40mm_HandSolder, symbol Device:R
- added R6, R7: 1.5k, Resistor_SMD:R_0805_2012Metric_Pad1.20x1.40mm_HandSolder, symbol Device:R
- added U1: BQ24074RGT, Package_DFN_QFN:VQFN-16-1EP_3x3mm_P0.5mm_EP1.6x1.6mm, symbol Battery_Management:BQ24074RGT
- added U2: LD1117S33TR_SOT223, Package_TO_SOT_SMD:SOT-223-3_TabPin2, symbol Regulator_Linear:LD1117S33TR_SOT223
- C3: renamed from C?; value 10uf -> 10u; footprint (none) -> Capacitor_SMD:C_0805_2012Metric_Pad1.18x1.45mm_HandSolder
- C4: renamed from C?; value 0.1uf -> 0.1u; footprint (none) -> Capacitor_SMD:C_0805_2012Metric_Pad1.18x1.45mm_HandSolder
- D5: renamed from D?; footprint (none) -> Diode_SMD:D_SOD-123F
- D6, D7: renamed from D?; footprint (none) -> LED_SMD:LED_0805_2012Metric_Pad1.15x1.40mm_HandSolder
- FB1: renamed from FB?; footprint (none) -> Resistor_SMD:R_0805_2012Metric_Pad1.20x1.40mm_HandSolder
- J1: renamed from J?; footprint (none) -> Connector_USB:USB_C_Receptacle_HRO_TYPE-C-31-M-12
- R4, R5: renamed from R?; footprint (none) -> Resistor_SMD:R_0805_2012Metric_Pad1.20x1.40mm_HandSolder
- R8: renamed from R?; value 300 -> 1.5k; footprint (none) -> Resistor_SMD:R_0805_2012Metric_Pad1.20x1.40mm_HandSolder
- R9: renamed from R?; value 150 -> 300; footprint (none) -> Resistor_SMD:R_0805_2012Metric_Pad1.20x1.40mm_HandSolder
- gave numbers to parts that had none: 2
Connections:
- net +3V3: now also C6.2, U2.2 (VO)
- net +5V: now also C1.2, U1.13 (IN)
- net GND: now also C1.1, C2.2, C5.2, C6.1, J2.3 (Pin_3), R1.2, R2.2, R3.2, U1.14 (TMR), U1.17 (VSS), U1.4 (~{CE}), U1.6 (EN1), U1.8 (VSS), U2.1 (GND)
- net USB_PWR_IN renamed VBUS
- new net: R3.1, U1.16 (ISET)
- new net: D4.1 (K), U1.9 (~{CHG})
- new net: D4.2 (A), R7.2
- new net: J2.1 (Pin_1), U1.2 (BAT), U1.3 (BAT)
- new net: J2.2 (Pin_2), U1.1 (TS)
- new net: R2.1, U1.12 (ILIM)
- new net: R1.1, U1.15 (ITERM)
- new net: D3.2 (A), R6.2
- new net: D3.1 (K), U1.7 (~{PGOOD})
- new net 5V_MASTER: C2.1, C5.1, R6.1, R7.1, U1.10 (OUT), U1.11 (OUT), U1.5 (EN2), U2.3 (VI)
Other:
- note added: "Battery Charger and Power Path Circuit"
- note added: "LDO 5V to 3.3V"
- moved on the sheet: C3, C4, D5, D6, D7, FB1, R8, R9
